File: Hardware/Electronic/SMACAR MAIN BOARD/SMACAR MAIN BOARD.kicad_pcb (KiCad board)
At the start: 2 copper layers, 14 parts, among them J2 Conn_01x02, U2 ESP32-S3-DevKitC

Commit message: aaaa
Parts:
- MOLEX1: value ELECTRICAL CONDUCTIVITY SENSOR -> EC
- MOLEX2: value M03PTH -> PH
- MOLEX3: value M03PTH -> TDS
- MOLEX5: value M04PTH -> LORAWAN
Other:
- board outline added: 60.5 x 71 mm
Changed lines of the file:
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@@
 			)
 		)
-		(property "Value" "M04PTH"
+		(property "Value" "LORAWAN"
 			(at 3.81 4.08 90)
 			(layer "F.SilkS")
@@
 			)
 		)
-		(property "Value" "M03PTH"
+		(property "Value" "PH"
 			(at 3.39 4.2 90)
 			(layer "F.SilkS")
@@
 			)
 		)
-		(property "Value" "ELECTRICAL CONDUCTIVITY SENSOR"
-			(at 9.04 4.25 90)
+		(property "Value" "EC"
+			(at 2.79 4.25 90)
 			(layer "F.SilkS")
 			(effects
@@
 			)
 		)
-		(property "Value" "M03PTH"
+		(property "Value" "TDS"
 			(at 2.54 4.08 90)
 			(layer "F.SilkS")
@@
 		)
 	)
+	(gr_rect
+		(start 101.5 30.5)
+		(end 162 101.5)
+		(stroke
+			(width 0.05)
+			(type default)
+		)
+		(fill no)
+		(layer "Edge.Cuts")
+	)
 	(gr_text "MAIN BOARD SMACAR"
