File: Hardware/Electronic/SMACAR MAIN BOARD/SMACAR MAIN BOARD/SMACAR MAIN BOARD.kicad_pcb (KiCad board)
At the start: 2 copper layers, 60.5 x 72.5 mm, 14 parts, among them J2 Conn_01x02, U2 ESP32-S3-DevKitC

Commit message: Hola
Routing:
- added copper zone on B.Cu, net GND
Changed lines of the file:
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@@
 		(net 38)
+	)
+	(zone
+		(net 1)
+		(net_name "GND")
+		(layer "B.Cu")
+		(hatch edge 0.5)
+		(connect_pads
+			(clearance 0.5)
+		)
+		(min_thickness 0.25)
+		(filled_areas_thickness no)
+		(fill
+			(thermal_gap 0.5)
+			(thermal_bridge_width 0.5)
+		)
+		(polygon
+			(pts
+				(xy 101.5 28.5) (xy 161.552979 28.5) (xy 162.035263 101.324916) (xy 101.5 101.817073)
+			)
+		)
 	)
 	(embedded_fonts no)
